Commit message: 烂完了

File: src/yeahbot_c1/urdf/yeahbot_c1.urdf (robot description, URDF)
Before this commit: robot yeahbot_c1, 20 links, 19 joints
Joints:
- joint arm_5_1_joint: axis 0.999181086402419 0.0404617165518926 -7.79060685413583E-05 -> (none); limit lower=-1.57 upper=1.57 effort=100 velocity=1 -> (none); type revolute -> fixed
- joint arm_5_2_joint: axis -0.999181086402419 -0.0404617165519045 7.79060685561991E-05 -> (none); limit lower=-1.57 upper=1.57 effort=100 velocity=1 -> (none); type revolute -> fixed
- joint arm_5_3_joint: axis 0.999181086402419 0.0404617165519009 -7.79060685332649E-05 -> (none); limit lower=-1.57 upper=1.57 effort=100 velocity=0 -> (none); type revolute -> fixed
- joint arm_5_4_joint: axis -0.999181086402419 -0.0404617165518986 7.79060685375041E-05 -> (none); limit lower=-1.57 upper=1.57 effort=100 velocity=1 -> (none); type revolute -> fixed
- joint arm_5_5_joint: axis 0.999181086402419 0.0404617165519009 -7.79060685332649E-05 -> (none); limit lower=-1.57 upper=1.57 effort=100 velocity=1 -> (none); type revolute -> fixed
- joint arm_5_6_joint: axis 0.999181086402419 0.0404617165519009 -7.79060685332649E-05 -> (none); limit lower=-1.57 upper=1.57 effort=100 velocity=1 -> (none); type revolute -> fixed
- joint wheel_lb_joint: axis 0 1 0 -> (none); type continuous -> fixed
- joint wheel_lf_joint: axis 0 1 0 -> (none); type continuous -> fixed
- joint wheel_rb_joint: axis 0 1 0 -> (none); type continuous -> fixed
- joint wheel_rf_joint: axis 0 1 0 -> (none); type continuous -> fixed
